Commit message: Update sensors.xacro

File: src/mecanum_description/urdf/sensors.xacro (robot description, xacro)
@@ -90,5 +90,5 @@
     <origin xyz="0 0 -0.038" rpy="0 3.1416 0"/>  <!-- facing down -->
   </joint>
-  <!-- ── TCRT5000 line tracker — front-centre bottom (on Arduino) ──────── -->
+  <!-- ── TCRT5000 line tracker — front-centre bottom (on Teensy 2) ──────── -->
   <link name="line_tracker_link"/>
   <joint name="line_tracker_joint" type="fixed">
@@ -97,3 +97,33 @@
     <origin xyz="0.080 0 -0.038" rpy="0 3.1416 0"/>  <!-- facing down, front biased -->
   </joint>
+  <!-- ── Plank A — extends left for crater loop object knock ───────────── -->
+  <!-- Physical: horizontal arm at 90°, sweeps at body height              -->
+  <link name="plank_a_link"/>
+  <joint name="plank_a_joint" type="fixed">
+    <parent link="base_link"/>
+    <child  link="plank_a_link"/>
+    <origin xyz="0 0.089 0.020" rpy="0 0 1.5708"/>  <!-- ⚠️ update when measured -->
+  </joint>
+  <!-- ── Plank B — lifts RGB sensor + IR transmitter to read antenna LEDs  -->
+  <!-- Two positions: 90° (low antennas) and 150° (high antennas)          -->
+  <link name="plank_b_link"/>
+  <joint name="plank_b_joint" type="fixed">
+    <parent link="base_link"/>
+    <child  link="plank_b_link"/>
+    <origin xyz="0.060 0 0.038" rpy="0 0 0"/>  <!-- ⚠️ update when measured -->
+  </joint>
+  <!-- ── RGB sensor (TCS34725) — mounted on tip of Plank B ─────────────── -->
+  <link name="rgb_sensor_link"/>
+  <joint name="rgb_sensor_joint" type="fixed">
+    <parent link="plank_b_link"/>
+    <child  link="rgb_sensor_link"/>
+    <origin xyz="0.100 0 0" rpy="0 0 0"/>  <!-- tip of plank B, facing forward -->
+  </joint>
+  <!-- ── IR transmitter — mounted on tip of Plank B beside RGB sensor ───── -->
+  <link name="ir_transmitter_link"/>
+  <joint name="ir_transmitter_joint" type="fixed">
+    <parent link="plank_b_link"/>
+    <child  link="ir_transmitter_link"/>
+    <origin xyz="0.100 0.020 0" rpy="0 0 0"/>  <!-- beside RGB sensor -->
+  </joint>
 </robot>

Commit message: Update sensors.xacro

File: src/mecanum_description/urdf/sensors.xacro (robot description, xacro)
@@ -12,6 +12,6 @@
       Ultrasonic RL  — rear-left corner
       Ultrasonic RR  — rear-right corner
-    RIGHT SIDE of robot (-y direction):
-      ToF 2 (side)   — right side centre (antenna_2 strafe + crank)
+    LEFT SIDE of robot (+y direction):
+      ToF 2 (side)   — left side centre (antenna_2 crank approach)
     BOTTOM (facing down):
       Optical flow   — centre underside
@@ -48,10 +48,10 @@
     <origin xyz="-0.127 -0.040 0" rpy="0 0 3.1416"/>  <!-- facing rear -->
   </joint>
-  <!-- ── ToF sensor 2 — RIGHT SIDE (antenna_2 strafe + crank) ─────────── -->
+  <!-- ── ToF sensor 2 — LEFT SIDE (antenna_2 crank approach) ──────────── -->
   <link name="tof_2_link"/>
   <joint name="tof_2_joint" type="fixed">
     <parent link="base_link"/>
     <child  link="tof_2_link"/>
-    <origin xyz="0 -0.089 0" rpy="0 0 -1.5708"/>  <!-- facing right -->
+    <origin xyz="0 0.089 0" rpy="0 0 1.5708"/>  <!-- facing left -->
   </joint>
   <!-- ── Ultrasonic FL — front-left ───────────────────────────────────── -->
@@ -97,5 +97,5 @@
     <origin xyz="0.080 0 -0.038" rpy="0 3.1416 0"/>  <!-- facing down, front biased -->
   </joint>
-  <!-- ── Plank A — extends left for crater loop object knock ───────────── -->
+  <!-- ── Plank A — physical arm on robot (not used in current mission) ──────── -->
   <!-- Physical: horizontal arm at 90°, sweeps at body height              -->
   <link name="plank_a_link"/>
